Commit message: Changed mesh paths for panda

File: urdfs/robots/franka_panda/panda.urdf (robot description, URDF)
Before this commit: robot panda, 14 links, 13 joints
Links:
- link panda_hand: geometry collision mesh filename=package://robot_assets/robots/franka_panda/hand.stl; visual mesh filename=package://robot_assets/robots/franka_panda/hand.dae
- link panda_leftfinger: geometry collision mesh filename=package://robot_assets/robots/franka_panda/finger.stl; visual mesh filename=package://robot_assets/robots/franka_panda/finger.dae
- link panda_link0: geometry collision mesh filename=package://robot_assets/robots/franka_panda/link0.stl; visual mesh filename=package://robot_assets/robots/franka_panda/link0.dae
- link panda_link1: geometry collision mesh filename=package://robot_assets/robots/franka_panda/link1.stl; visual mesh filename=package://robot_assets/robots/franka_panda/link1.dae
- link panda_link2: geometry collision mesh filename=package://robot_assets/robots/franka_panda/link2.stl; visual mesh filename=package://robot_assets/robots/franka_panda/link2.dae
- link panda_link3: geometry collision mesh filename=package://robot_assets/robots/franka_panda/link3.stl; visual mesh filename=package://robot_assets/robots/franka_panda/link3.dae
- link panda_link4: geometry collision mesh filename=package://robot_assets/robots/franka_panda/link4.stl; visual mesh filename=package://robot_assets/robots/franka_panda/link4.dae
- link panda_link5: geometry collision mesh filename=package://robot_assets/robots/franka_panda/link5.stl; visual mesh filename=package://robot_assets/robots/franka_panda/link5.dae
- link panda_link6: geometry collision mesh filename=package://robot_assets/robots/franka_panda/link6.stl; visual mesh filename=package://robot_assets/robots/franka_panda/link6.dae
- link panda_link7: geometry collision mesh filename=package://robot_assets/robots/franka_panda/link7.stl; visual mesh filename=package://robot_assets/robots/franka_panda/link7.dae
- link panda_rightfinger: geometry collision mesh filename=package://robot_assets/robots/franka_panda/finger.stl; visual mesh filename=package://robot_assets/robots/franka_panda/finger.dae
