Commit message: Modified urdfs for panda and kinova

File: urdfs/robots/kinova/kinova.urdf (robot description, URDF)
Before this commit: robot kinova, 15 links, 14 joints
Links:
- link j2s6s200_link_1: geometry collision mesh filename=package://robot_assets/robots/kinova/shoulder.dae; visual mesh filename=package://robot_assets/robots/kinova/ring_big.dae
- link j2s6s200_link_2: geometry collision mesh filename=package://robot_assets/robots/kinova/arm.dae; visual mesh filename=package://robot_assets/robots/kinova/arm.dae
- link j2s6s200_link_3: geometry collision mesh filename=package://robot_assets/robots/kinova/forearm.dae; visual mesh filename=package://robot_assets/robots/kinova/forearm.dae
- link j2s6s200_link_4: geometry collision mesh filename=package://robot_assets/robots/kinova/wrist_spherical_1.dae; visual mesh filename=package://robot_assets/robots/kinova/ring_small.dae
- link j2s6s200_link_5: geometry collision mesh filename=package://robot_assets/robots/kinova/wrist_spherical_2.dae; visual mesh filename=package://robot_assets/robots/kinova/ring_small.dae
- link j2s6s200_link_6: geometry collision mesh filename=package://robot_assets/robots/kinova/hand_2finger.dae; visual mesh filename=package://robot_assets/robots/kinova/hand_2finger.dae
- link j2s6s200_link_base: geometry collision mesh filename=package://robot_assets/robots/kinova/base.dae; visual mesh filename=package://robot_assets/robots/kinova/base.dae
- link j2s6s200_link_finger_1: geometry collision mesh filename=package://robot_assets/robots/kinova/finger_proximal.dae; visual mesh filename=package://robot_assets/robots/kinova/finger_proximal.dae
- link j2s6s200_link_finger_2: geometry collision mesh filename=package://robot_assets/robots/kinova/finger_proximal.dae; visual mesh filename=package://robot_assets/robots/kinova/finger_proximal.dae
- link j2s6s200_link_finger_tip_1: geometry collision mesh filename=package://robot_assets/robots/kinova/finger_distal.dae; visual mesh filename=package://robot_assets/robots/kinova/finger_distal.dae
- link j2s6s200_link_finger_tip_2: geometry collision mesh filename=package://robot_assets/robots/kinova/finger_distal.dae; visual mesh filename=package://robot_assets/robots/kinova/finger_distal.dae
- link jaco_front_hatch_support_v2: geometry visual mesh filename=package://robot_assets/robots/kinova/jaco_front_hatch_suppo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
- link jaco_mounting_block: geometry visual mesh filename=package://robot_assets/robots/kinova/jaco_mounting_block.dae
Joints:
- joint j2s6s200_joint_end_effector: limit lower=0 upper=0 effort=2000 velocity=1 -> lower=0 upper=0 effort=2000 velocity=0.99
- joint j2s6s200_joint_finger_1: limit lower=0 upper=1.51 effort=2 velocity=1 -> lower=0 upper=1.51 effort=2 velocity=0.99; type fixed -> revolute
- joint j2s6s200_joint_finger_2: limit lower=0 upper=1.51 effort=2 velocity=1 -> lower=0 upper=1.51 effort=2 velocity=0.99; type fixed -> revolute
- joint j2s6s200_joint_finger_tip_1: limit lower=0 upper=2 effort=2 velocity=1 -> lower=0 upper=2 effort=2 velocity=0.99
- joint j2s6s200_joint_finger_tip_2: limit lower=0 upper=2 effort=2 velocity=1 -> lower=0 upper=2 effort=2 velocity=0.99
